Commit message: add in msg and use xacro

File: ff_viz/model/ff.urdf.xacro (robot description, xacro)
@@ -1,8 +1,9 @@
 <?xml version="1.0"?>
-<robot name="ff">
+<robot xmlns:xacro="http://www.ros.org/wiki/xacro" name="ff">
   <material name="white">
     <color rgba="1 1 1 1"/>
   </material>
-  <link name="robot/base">
+  <xacro:arg name="robot_name" default="robot" />
+  <link name="$(arg robot_name)/base">
     <visual>
       <origin xyz="0 0 -0.12" rpy="1.570796327 0 0" />
